Commit message: Added data from calcs

File: bffv1_description/urdf/base.xacro (robot description, xacro)
@@ -20,11 +20,16 @@
 <!--  <xacro:property name="mass" value="6.25"/>-->
   <!-- Describing the dimensions of the vehicle's bounding box: width, length, height -->
+  <!-- BLUEROV2 -->
+  <!--
   <xacro:property name="x_size" value="0.448"/>
   <xacro:property name="y_size" value="0.2384"/>
   <xacro:property name="z_size" value="0.28066"/>
-  <!-- minion_usv_height is not really! It's just for run... We need first calculate the Fossen parameters -->
-  <!-- Volume -->
-  <xacro:property name="volume" value="0.011054"/>
-<!--  <xacro:property name="volume" value="0.00625"/>-->
+  -->
+  <!-- Float -->
+  <xacro:property name="x_size" value="0.106"/>
+  <xacro:property name="y_size" value="0.106"/>
+  <xacro:property name="z_size" value="0.6"/>
+  <!-- <xacro:property name="volume" value="0.011054"/> --> <!-- BLUEROV2 -->
+  <xacro:property name="volume" value="0.00625"/>
   <xacro:property name="cog" value="0 0 0"/>
   <xacro:property name="cob" value="0 0 0"/>
@@ -50,19 +55,21 @@
           otherwise your model will become unstable on Gazebo
         -->
+        <!-- From basic cylinder-->
+        <inertial>
+          <mass value="${mass}" />
+          <origin xyz="${cog}" rpy="0 0 0"/>
+          <inertia ixx="0.19153225" ixy="0" ixz="0"
+                   iyy="0.19153225" iyz="0"
+                   izz="0.0080645" />
+        </inertial>
+        <!-- BLUEROV2-->
 <!--        <inertial>-->
 <!--          <mass value="${mass}" />-->
 <!--          <origin xyz="${cog}" rpy="0 0 0"/>-->
-<!--          <inertia ixx="0.19153225" ixy="0" ixz="0"-->
-<!--                   iyy="0.19153225" iyz="0"-->
-<!--                   izz="0.0080645" />-->
+<!--          <inertia-->
+<!--                  ixx="${0.2*mass*y_size*y_size + 0.2*mass*z_size*z_size}" ixy="0.0" ixz="0.0"-->
+<!--                  iyy="${0.2*mass*x_size*x_size + 0.2*mass*z_size*z_size}" iyz="0.0"-->
+<!--                  izz="${0.2*mass*x_size*x_size + 0.2*mass*y_size*y_size}" />-->
 <!--        </inertial>-->
-        <inertial>
-          <mass value="${mass}" />
-          <origin xyz="${cog}" rpy="0 0 0"/>
-          <inertia
-                  ixx="${0.2*mass*y_size*y_size + 0.2*mass*z_size*z_size}" ixy="0.0" ixz="0.0"
-                  iyy="${0.2*mass*x_size*x_size + 0.2*mass*z_size*z_size}" iyz="0.0"
-                  izz="${0.2*mass*x_size*x_size + 0.2*mass*y_size*y_size}" />
-        </inertial>
         <visual>
           <origin xyz="0 0 0" rpy="0 0 0"/>

File: bffv1_description/urdf/gazebo.xacro (robot description, xacro)
@@ -61,4 +61,6 @@
           <type>fossen</type>
           <!-- Added mass: see p.28 in Berg2012 -->
+              <!-- BLUEROV2 -->
+              <!--
           <added_mass>
               1.7182 0 0 0 0 0
@@ -75,5 +77,21 @@
               0 0 0 0 0 0
           </quadratic_damping>
-          </hydrodynamic_model>
+          -->
+          <!-- From Calcs -->
+          <added_mass>
+              0 0 0 0 0 0
+              0 0 0 0 0 0
+              0 0 3.68 0 0 0
+              0 0 0 0.175 0 0
+              0 0 0 0 0.175 0
+              0 0 0 0 0 0.0
+          </added_mass>
+          <linear_damping>
+              -0.1 -0.1 -0.1 -0.1 -0.1 -0.1
+          </linear_damping>
+          <quadratic_damping>
+              0 0 0 0 0 0
+          </quadratic_damping>
+        </hydrodynamic_model>
       </link>
     </xacro:macro>

Commit message: Increased the linear damping to -5.0 to make it stable

File: bffv1_description/urdf/base.xacro (robot description, xacro)
@@ -17,6 +17,6 @@
   <!-- Fluid density -->
 <!--  <xacro:property name="rho" value="1028"/>-->
-  <xacro:property name="mass" value="11.38"/>
-<!--  <xacro:property name="mass" value="6.25"/>-->
+<!--  <xacro:property name="mass" value="11.38"/>-->
+  <xacro:property name="mass" value="6.25"/>
   <!-- Describing the dimensions of the vehicle's bounding box: width, length, height -->
   <!-- BLUEROV2 -->

File: bffv1_description/urdf/gazebo.xacro (robot description, xacro)
@@ -88,5 +88,5 @@
           </added_mass>
           <linear_damping>
-              -0.1 -0.1 -0.1 -0.1 -0.1 -0.1
+              -5.0 -5.0 -5.0 -5.0 -5.0 -5.0
           </linear_damping>
           <quadratic_damping>
